File: kicad/esr_stm32f030f4.kicad_sch (KiCad schematic)
At the start: 28 parts, among them J1 ESR, J2 SWD, SW1 power, U1 STM32F030F4Px, U2 MCP6001, U3 74LVC1G3157

Commit message: minor changes
Other:
- note added: "0.034"
- note added: "1/2"
- note added: "120 kHz"
- note added: "81-82@120k"
- note removed: "0.036"
- note removed: "120 kHz 1.2 kHz"
- moved on the sheet: R2
Changed lines of the file:
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@@
     (rev "1.5")
     (company "vadim_d, ozforester")
-    (comment 1 "cqham.ru/forum/xxx")
+    (comment 1 "http://www.cqham.ru/forum/showthread.php?47207")
+    (comment 2 "CC-BY-SA 4.0 License")
   )
   (junction (at 141.605 130.81) (diameter 0) (color 0 0 0 0)
@@
     (stroke (width 0) (type default) (color 0 0 0 1))
   )
-  (wire (pts (xy 132.715 120.65) (xy 135.255 120.65))
+  (wire (pts (xy 132.08 120.65) (xy 135.255 120.65))
     (stroke (width 0) (type default))
   )
@@
     (stroke (width 0) (type default))
   )
-  (wire (pts (xy 191.77 100.965) (xy 191.77 102.235))
-    (stroke (width 0) (type default))
-  )
   (wire (pts (xy 100.965 62.865) (xy 101.6 62.865))
     (stroke (width 0) (type default))
@@
     (stroke (width 0) (type default))
   )
-  (text "120 kHz\n1.2 kHz" (at 105.41 99.06 0)
+  (text "1/2" (at 158.75 104.14 0)
     (effects (font (size 1.27 1.27)) (justify left bottom))
   )
-  (text "0.036" (at 165.735 100.965 0)
+  (text "120 kHz" (at 123.825 91.44 0)
+    (effects (font (size 1.27 1.27)) (justify left bottom))
+  )
+  (text "0.034" (at 165.735 100.965 0)
     (effects (font (size 1.27 1.27)) (justify left bottom))
   )
@@
     (effects (font (size 1.27 1.27)) (justify left bottom))
   )
+  (text "81-82@120k" (at 136.525 54.61 0)
+    (effects (font (size 1.27 1.27)) (justify left bottom))
+  )
   (text "TIM1CH3" (at 105.41 94.615 0)
+    (effects (font (size 1.27 1.27)) (justify left bottom))
+  )
+  (text "1/2" (at 186.055 112.395 0)
     (effects (font (size 1.27 1.27)) (justify left bottom))
   )
@@
     )
   )
-  (symbol (lib_id "power:VCC") (at 132.715 113.03 0) (unit 1)
-    (in_bom yes) (on_board yes) (dnp no)
-    (property "Reference" "#PWR08" (at 132.715 116.84 0)
-      (effects (font (size 1.27 1.27)) hide)
-    )
-    (property "Value" "3v" (at 131.445 109.22 0)
-      (effects (font (size 1.27 1.27)) (justify left))
-    )
-    (property "Footprint" "" (at 132.715 113.03 0)
-      (effects (font (size 1.27 1.27)) hide)
-    )
-    (property "Datasheet" "" (at 132.715 113.03 0)
+  (symbol (lib_id "power:VCC") (at 132.08 113.03 0) (unit 1)
+    (in_bom yes) (on_board yes) (dnp no)
+    (property "Reference" "#PWR08" (at 132.08 116.84 0)
+      (effects (font (size 1.27 1.27)) hide)
+    )
+    (property "Value" "3v" (at 130.81 109.22 0)
+      (effects (font (size 1.27 1.27)) (justify left))
+    )
+    (property "Footprint" "" (at 132.08 113.03 0)
+      (effects (font (size 1.27 1.27)) hide)
+    )
+    (property "Datasheet" "" (at 132.08 113.03 0)
       (effects (font (size 1.27 1.27)) hide)
     )
@@
     )
   )
-  (symbol (lib_id "Device:R") (at 132.715 116.84 0) (unit 1)
-    (in_bom yes) (on_board yes) (dnp no)
-    (property "Reference" "R2" (at 127.635 113.665 0)
-      (effects (font (size 1.27 1.27)) (justify left))
-    )
-    (property "Value" "10k" (at 127 116.205 0)
-      (effects (font (size 1.27 1.27)) (justify left))
-    )
-    (property "Footprint" "Resistor_SMD:R_0805_2012Metric" (at 130.937 116.84 90)
-      (effects (font (size 1.27 1.27)) hide)
-    )
-    (property "Datasheet" "~" (at 132.715 116.84 0)
+  (symbol (lib_id "Device:R") (at 132.08 116.84 0) (unit 1)
+    (in_bom yes) (on_board yes) (dnp no)
+    (property "Reference" "R2" (at 127 113.665 0)
+      (effects (font (size 1.27 1.27)) (justify left))
+    )
+    (property "Value" "10k" (at 126.365 116.205 0)
+      (effects (font (size 1.27 1.27)) (justify left))
+    )
+    (property "Footprint" "Resistor_SMD:R_0805_2012Metric" (at 130.302 116.84 90)
+      (effects (font (size 1.27 1.27)) hide)
+    )
+    (property "Datasheet" "~" (at 132.08 116.84 0)
       (effects (font (size 1.27 1.27)) hide)
     )
@@
     )
   )
-  (symbol (lib_id "power:GND") (at 191.77 102.235 90) (unit 1)
-    (in_bom yes) (on_board yes) (dnp no)
-    (property "Reference" "#PWR024" (at 198.12 102.235 0)
-      (effects (font (size 1.27 1.27)) hide)
-    )
-    (property "Value" "GND" (at 196.1642 102.108 0)
-      (effects (font (size 1.27 1.27)) hide)
-    )
-    (property "Footprint" "" (at 191.77 102.235 0)
-      (effects (font (size 1.27 1.27)) hide)
-    )
-    (property "Datasheet" "" (at 191.77 102.235 0)
+  (symbol (lib_id "power:GND") (at 191.77 100.965 90) (unit 1)
+    (in_bom yes) (on_board yes) (dnp no)
+    (property "Reference" "#PWR024" (at 198.12 100.965 0)
+      (effects (font (size 1.27 1.27)) hide)
+    )
+    (property "Value" "GND" (at 196.1642 100.838 0)
+      (effects (font (size 1.27 1.27)) hide)
+    )
+    (property "Footprint" "" (at 191.77 100.965 0)
+      (effects (font (size 1.27 1.27)) hide)
+    )
+    (property "Datasheet" "" (at 191.77 100.965 0)
       (effects (font (size 1.27 1.27)) hide)
     )
@@
   (symbol (lib_id "MCU_ST_STM32F0:STM32F030F4Px") (at 109.22 86.36 0) (unit 1)
     (in_bom yes) (on_board yes) (dnp no)
-    (property "Reference" "U1" (at 112.395 110.49 0)
-      (effects (font (size 1.27 1.27)) (justify left))
-    )
-    (property "Value" "STM32F030F4Px" (at 105.41 113.03 0)
+    (property "Reference" "U1" (at 111.76 111.125 0)
+      (effects (font (size 1.27 1.27)) (justify left))
+    )
+    (property "Value" "STM32F030F4Px" (at 102.87 113.665 0)
       (effects (font (size 1.27 1.27)) (justify left))
     )
@@
   (symbol (lib_id "Connector:Conn_01x02_Pin") (at 127 99.06 180) (unit 1)
     (in_bom yes) (on_board yes) (dnp no)
-    (property "Reference" "J2" (at 128.905 97.155 0)
+    (property "Reference" "J2" (at 128.7259 96.5685 0)
       (effects (font (size 1.27 1.27)) (justify right))
     )
-    (property "Value" "SWD" (at 128.27 99.695 0)
+    (property "Value" "SWD" (at 127.8901 98.7175 0)
       (effects (font (size 1.27 1.27)) (justify right))
     )
